File: corne-classic/pcb/corne-classic.kicad_pcb (KiCad board)
At the start: 2 copper layers, 133.8 x 111.2 mm, 117 parts, among them J1 MJ-4PP-9, J2 OLED, J3 LED, P1 i2c-pin, P2 i2c-pin, SW1 SW_PUSH, SW10 SW_PUSH, SW11 SW_PUSH, SW12 SW_PUSH, SW13 SW_PUSH, SW14 SW_PUSH, SW15 SW_PUSH, SW16 SW_PUSH, SW17 SW_PUSH, SW18 SW_PUSH, SW19 SW_PUSH, SW2 SW_PUSH, SW20 SW_PUSH, SW21 SW_PUSH, SW22 SW_PUSH, SW23 SW_PUSH, SW24 SW_PUSH, SW25 SW_PUSH, SW26 SW_PUSH, SW27 SW_PUSH, SW28 SW_PUSH, SW3 SW_PUSH, SW4 SW_PUSH, SW5 SW_PUSH, SW6 SW_PUSH, SW7 SW_PUSH, SW8 SW_PUSH, SW9 SW_PUSH, U1 ProMicro

Commit message: logo added
Parts:
- added G***: LOGO, kbd:sing_w_1500, F.Cu at (183.7, 112.3)
- added G***: LOGO, kbd:sing_t1_900, F.Cu at (184.4, 120.8)
- added G***: LOGO, kbd:sing_w_reverse_1500, F.Cu at (183.7, 112.3)
- added G***: LOGO, kbd:sing_t1_reverse_900, F.Cu at (184.4, 120.8)
Other:
- board text added: "v1.0 by XWaVeX"
- board text removed: "corne-ext designed by XWaVeX"

Commit message: restructuring
Parts:
- added L0: SK6812MINI, kbd:SK6812MINI_underglow_rev, F.Cu at (165.0, 64.9)
- added L111: SK6812MINI, kbd:SK6812MINI_underglow_rev, F.Cu at (89.0, 67.3)
- RSW1: value Reset -> SW_PUSH
Connections:
- L2 pad 1: Net-(L1-Pad3) -> Net-(L111-Pad3)
- L3 pad 3: LED -> Net-(L0-Pad1)
Routing:
- net Net-(L111-Pad3): track 0.00 -> 53.0 mm, vias 0 -> 3
- net Net-(L0-Pad1): track 0.00 -> 43.4 mm, vias 0 -> 6
- net GND: track 980.2 -> 1008.5 mm, vias 157 -> 52
- net Net-(L12-Pad3): track 38.6 -> 53.5 mm, vias 4 -> 8
- net VCC: track 976.4 -> 988.4 mm, vias 45 -> 50
- net Net-(L1-Pad3): track 45.4 -> 52.8 mm, vias 5 -> 6
- net col3: track 240.8 -> 247.9 mm, vias 6 -> 8
- net Net-(L14-Pad1): track 36.5 -> 43.4 mm, vias 4 -> 6
- net col1: track 253.1 -> 251.3 mm
- net LED: track 70.9 -> 69.2 mm
- net col5: track 212.5 -> 211.6 mm
- net SCL: track 47.9 -> 48.7 mm
- net Net-(L18-Pad3): track 40.3 -> 40.9 mm
- net (no net): vias 4 -> 0

Commit message: final?
Parts:
- removed the G*** at (183.7, 112.3) (x2)
- removed the G*** at (184.4, 120.8) (x2)
- added G***: LOGO, kbd:sing_t1_solder_900, B.Cu at (184.4, 122.0)
- added G***: LOGO, kbd:sing_w_solder_1500, B.Cu at (183.7, 113.7)
- added G***: LOGO, kbd:sing_w_solder_1500, F.Cu at (183.7, 113.7)
- added G***: LOGO, kbd:sing_t1_solder_900, F.Cu at (184.4, 122.0)
- moved ? 1.45 mm to (192.2, 112.8)
- moved ? 1.45 mm to (177.8, 104.3)
Routing:
- net VCC: track 988.4 -> 984.6 mm
- net Net-(L34-Pad3): track 40.5 -> 38.5 mm
- net GND: track 1008.5 -> 1009.4 mm
Other:
- board text added: "based on crkbd v2.0 by foostan"

Commit message: included all gerber files
Routing:
- net GND: track 1009.4 -> 1010.8 mm
